File: hardware/REV2_SPRING_2022/REV2_SPRING_2022.sch (KiCad schematic (older format))
At the start: 40 parts, among them J101 Screw_Terminal_01x02, J102 Screw_Terminal_01x02, J103 Conn_01x02_Female, J104 Screw_Terminal_01x02, J105 Conn_01x02_Female, J107 Screw_Terminal_01x02, J109 Conn_01x02_Female, J110 Conn_01x02_Female, Q101 Q_NMOS_GDS, Q102 Q_NMOS_GDS, U1 Teensy3.6_All_Pins, U2 PA16165_Breakout, U3 MPL3115A2_Breakout, U4 BNO055_Breakout, U5 RFM69HCW_Breakout

Commit message: File structure update
Parts:
- U2: symbol Sensors_2021_2022:PA16165_Breakout -> REV2_SPRING_2022-rescue:PA16165_Breakout-Sensors_2021_2022
- U3: symbol Sensors_2021_2022:MPL3115A2_Breakout -> REV2_SPRING_2022-rescue:MPL3115A2_Breakout-Sensors_2021_2022
- U4: symbol Sensors_2021_2022:BNO055_Breakout -> REV2_SPRING_2022-rescue:BNO055_Breakout-Sensors_2021_2022
- U5: symbol Sensors_2021_2022:RFM69HCW_Breakout -> REV2_SPRING_2022-rescue:RFM69HCW_Breakout-Sensors_2021_2022
Changed lines of the file:
@@
 $EndComp
 $Comp
-L Sensors_2021_2022:BNO055_Breakout U4
+L REV2_SPRING_2022-rescue:BNO055_Breakout-Sensors_2021_2022 U4
 U 1 1 61992B5E
 P 5950 2000
@@
 $EndComp
 $Comp
-L Sensors_2021_2022:MPL3115A2_Breakout U3
+L REV2_SPRING_2022-rescue:MPL3115A2_Breakout-Sensors_2021_2022 U3
 U 1 1 61994643
 P 5900 3950
@@
 NoConn ~ 9400 1650
 $Comp
-L Sensors_2021_2022:RFM69HCW_Breakout U5
+L REV2_SPRING_2022-rescue:RFM69HCW_Breakout-Sensors_2021_2022 U5
 U 1 1 6194AAD4
 P 9050 2250
@@
 $EndComp
 $Comp
-L Sensors_2021_2022:PA16165_Breakout U2
+L REV2_SPRING_2022-rescue:PA16165_Breakout-Sensors_2021_2022 U2
 U 1 1 6199B8C8
 P 5850 6000
