File: hardware/REV2_SPRING_2022/TPS2113A_Teesny.sch (KiCad schematic (older format))
At the start: 7 parts, among them U201 TPS2113ADRBR

Commit message: File structure update
Parts:
- U201: symbol TPS2113ADRBR:TPS2113ADRBR -> REV2_SPRING_2022-rescue:TPS2113ADRBR-TPS2113ADRBR
Changed lines of the file:
@@
 $EndDescr
 $Comp
-L TPS2113ADRBR:TPS2113ADRBR U?
+L REV2_SPRING_2022-rescue:TPS2113ADRBR-TPS2113ADRBR U?
 U 1 1 61AB462E
 P 6600 3050
