File: hardware/REV2_SPRING_2022/REV2_SPRING_2022.kicad_sch (KiCad schematic)
At the start: 40 parts

Commit message: Reverse Current
Parts:
- BT101, BT102: value (none) -> Battery_Cell; footprint (none) -> Olin_Rocketry:MyBatteryHolder_MPD_BH-18650-PC2
- BZ101: value (none) -> Buzzer; footprint (none) -> Olin_Rocketry:Large_Buzzer_24mmOD_14.8mmPinDistance_1.0mmPinDiameter
- C101: value (none) -> C_0.1u; footprint (none) -> Capacitor_SMD:C_0805_2012Metric_Pad1.18x1.45mm_HandSolder
- D101, D102, D103, D104, D105, D106: value (none) -> LED; footprint (none) -> LED_SMD:LED_0805_2012Metric_Pad1.15x1.40mm_HandSolder
- J101, J102, J104, J107: value (none) -> Screw_Terminal_01x02; footprint (none) -> TerminalBlock:TerminalBlock_bornier-2_P5.08mm
- J103, J105, J109, J110: value (none) -> Conn_01x02_Female; footprint (none) -> Connector_Wire:SolderWire-1sqmm_1x02_P5.4mm_D1.4mm_OD2.7mm_Relief2x
- Q101, Q102: value (none) -> Q_NMOS_GDS; footprint (none) -> footprints:TO-220-3
- R101: value (none) -> R_15k; footprint (none) -> Resistor_SMD:R_0805_2012Metric_Pad1.20x1.40mm_HandSolder
- R102: value (none) -> R_4.7k; footprint (none) -> Resistor_SMD:R_0805_2012Metric_Pad1.20x1.40mm_HandSolder
- R103, R109, R110, R111, R112, R114, R115: value (none) -> R_10k; footprint (none) -> Resistor_SMD:R_0805_2012Metric_Pad1.20x1.40mm_HandSolder
- R104, R105, R106, R107, R108, R113: value (none) -> R_750; footprint (none) -> Resistor_SMD:R_0805_2012Metric_Pad1.20x1.40mm_HandSolder
- U1: value (none) -> Teensy3.6_All_Pins; footprint (none) -> teensy:Teensy35_36
- U2: value (none) -> PA16165_Breakout; footprint (none) -> sensors_2021_2022:PA16165_Breakout
- U3: value (none) -> MPL3115A2_Breakout; footprint (none) -> sensors_2021_2022:MPL3115A2_Breakout
- U4: value (none) -> BNO055_Breakout; footprint (none) -> sensors_2021_2022:BNO055_Breakout
- U5: value (none) -> RFM69HCW_Breakout; footprint (none) -> sensors_2021_2022:RFM69HCW_Breakout
