File: hardware/REV3_FALL_2023/PRISM_Teensy/board_one_teensy_22/board_one_teensy_22.kicad_sch (KiCad schematic)
At the start: 20 parts, among them J2 PRISM_IO_INTERFACE, J3 3387, U1 Teensy4.0, U2 GPS-14414, U3 3966, U4 RFM69HCW_Breakout

Commit message: Finished Schematic
Parts:
- removed J3: 3387, 3387, symbol LSM9DS1:3387
- added C3, C4, C6: C_100nF, footprints:C_0603_1608Metric, symbol formula:C_100nF
- added C5: C_10uF, footprints:C_0805_OEM, symbol formula:C_10uF
- added C7: C_10nF, footprints:C_1206_OEM, symbol formula:C_10nF
- added J1: Micro_SD_Card, symbol Connector:Micro_SD_Card
- added R1, R2, R3: R_10K, footprints:R_0805_OEM, symbol formula:R_10K
- added U5: LSM9DS1, Package_LGA:LGA-24L_3x3.5mm_P0.43mm, symbol Sensor_Motion:LSM9DS1
Connections:
- net 3.3V: now also C3.2, C4.2, C5.1, R1.1, R2.1, R3.1, U5.1 (VDDIO), U5.22 (VDD), U5.23 (VDD), U5.3 (VDDIO)
- net GND: now also C3.1, C4.1, C5.2, C6.2, C7.2, J1.6 (VSS), J1.9 (SHIELD), U5.14 (RES), U5.15 (RES), U5.16 (RES), U5.17 (RES), U5.18 (RES), U5.19 (GND), U5.20 (GND)
- net SCL 0: now also R1.2, U5.2 (SCL/SPC)
- net SDA 0: now also R2.2, U5.4 (SDA/SDI/SDO), U5.6 (SDO_M)
- new net: R3.2, U5.13 (DEN_A/G)
- new net: C7.1, U5.21 (CAP)
- new net: C6.1, U5.24 (C1)
- no-connect marks 32 -> 25
