File: hardware/MiniAvionics/Barometer.kicad_sch (KiCad schematic)
At the start: 7 parts, among them U1 BMP390

Commit message: Kicad
Parts:
- C1, C2: value 100nF -> 0.1uF; footprint (none) -> Resistor_SMD:R_0603_1608Metric
- GREEN1: footprint (none) -> Resistor_SMD:R_0603_1608Metric
- R1, R2: value 4700Ω -> 4.7k; footprint (none) -> Resistor_SMD:R_0603_1608Metric
- R3: value 10000Ω -> 10k; footprint (none) -> Resistor_SMD:R_0603_1608Metric
Changed lines of the file:
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@@
       (effects (font (size 1.27 1.27)) (justify right))
     )
-    (property "Footprint" "" (at 99.06 39.37 0)
+    (property "Footprint" "Resistor_SMD:R_0603_1608Metric" (at 99.06 39.37 0)
       (effects (font (size 1.27 1.27)) hide)
     )
@@
       (effects (font (size 1.27 1.27)))
     )
-    (property "Value" "100nF" (at 87.63 35.56 90)
-      (effects (font (size 1.27 1.27)))
-    )
-    (property "Footprint" "" (at 92.4052 39.37 0)
+    (property "Value" "0.1uF" (at 87.63 35.56 90)
+      (effects (font (size 1.27 1.27)))
+    )
+    (property "Footprint" "Resistor_SMD:R_0603_1608Metric" (at 92.4052 39.37 0)
       (effects (font (size 1.27 1.27)) hide)
     )
@@
       (effects (font (size 1.27 1.27)))
     )
-    (property "Value" "4700Ω" (at 36.83 38.1 90)
-      (effects (font (size 1.27 1.27)))
-    )
-    (property "Footprint" "" (at 36.83 37.338 90)
+    (property "Value" "4.7k" (at 36.83 38.1 90)
+      (effects (font (size 1.27 1.27)))
+    )
+    (property "Footprint" "Resistor_SMD:R_0603_1608Metric" (at 36.83 37.338 90)
       (effects (font (size 1.27 1.27)) hide)
     )
@@
       (effects (font (size 1.27 1.27)))
     )
-    (property "Value" "100nF" (at 22.86 41.91 90)
-      (effects (font (size 1.27 1.27)))
-    )
-    (property "Footprint" "" (at 27.6352 45.72 0)
+    (property "Value" "0.1uF" (at 22.86 41.91 90)
+      (effects (font (size 1.27 1.27)))
+    )
+    (property "Footprint" "Resistor_SMD:R_0603_1608Metric" (at 27.6352 45.72 0)
       (effects (font (size 1.27 1.27)) hide)
     )
@@
       (effects (font (size 1.27 1.27)) (justify left))
     )
-    (property "Value" "10000Ω" (at 101.6 35.56 90)
-      (effects (font (size 1.27 1.27)) (justify left))
-    )
-    (property "Footprint" "" (at 97.282 31.75 90)
+    (property "Value" "10k" (at 101.6 35.56 90)
+      (effects (font (size 1.27 1.27)) (justify left))
+    )
+    (property "Footprint" "Resistor_SMD:R_0603_1608Metric" (at 97.282 31.75 90)
       (effects (font (size 1.27 1.27)) hide)
     )
@@
       (effects (font (size 1.27 1.27)) (justify left))
     )
-    (property "Value" "4700Ω" (at 34.29 55.88 90)
-      (effects (font (size 1.27 1.27)) (justify left))
-    )
-    (property "Footprint" "" (at 29.972 52.07 90)
-      (effects (font (size 1.27 1.27)) hide)
-    )
+    (property "Value" "4.7k" (at 34.29 55.88 90)
+      (effects (font (size 1.27 1.27)) (justify left))
+    )
+    (property "Footprint" "Resistor_SMD:R_0603_1608Metric" (at 29.972 52.07 90)
+      (effects (font (size 1.27 1.27)) hide)
+    )

Commit message: bmp390
ff
Parts:
- U1: footprint LGA10_BMP390_BOS -> MiniAvionics:LGA10_BMP390_BOS
Changed lines of the file:
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@@
+    (effects (font (size 1.27 1.27)) (justify left bottom))
+  )
+  (label "VDDIO" (at 81.28 64.77 90) (fields_autoplaced)
     (effects (font (size 1.27 1.27)) (justify left bottom))
   )
@@
     )
   )
+  (symbol (lib_id "power:PWR_FLAG") (at 81.28 64.77 180) (unit 1)
+    (in_bom yes) (on_board yes) (dnp no) (fields_autoplaced)
+    (property "Reference" "#FLG02" (at 81.28 66.675 0)
+      (effects (font (size 1.27 1.27)) hide)
+    )
+    (property "Value" "PWR_FLAG" (at 81.28 69.85 0)
+      (effects (font (size 1.27 1.27)))
+    )
+    (property "Footprint" "" (at 81.28 64.77 0)
+      (effects (font (size 1.27 1.27)) hide)
+    )
+    (property "Datasheet" "~" (at 81.28 64.77 0)
+      (effects (font (size 1.27 1.27)) hide)
+    )
+    (pin "1")
+    (instances
+      (project "MiniAvionics"
+        (path "/db07439e-b2f9-4de9-a6da-003465a4a615/c809a2a1-09f7-4dc3-8e0e-630961f558de"
+          (reference "#FLG02") (unit 1)
+        )
+      )
+    )
+  )
   (symbol (lib_id "power:GND") (at 91.44 45.72 0) (unit 1)
     (in_bom yes) (on_board yes) (dnp no)
@@
     )
   )
+  (symbol (lib_id "power:GND") (at 72.39 67.31 0) (unit 1)
+    (in_bom yes) (on_board yes) (dnp no) (fields_autoplaced)
+    (property "Reference" "#PWR07" (at 72.39 73.66 0)
+      (effects (font (size 1.27 1.27)) hide)
+    )
+    (property "Value" "GND" (at 72.39 72.39 0)
+      (effects (font (size 1.27 1.27)))
+    )
+    (property "Footprint" "" (at 72.39 67.31 0)
+      (effects (font (size 1.27 1.27)) hide)
+    )
+    (property "Datasheet" "" (at 72.39 67.31 0)
+      (effects (font (size 1.27 1.27)) hide)
+    )
+    (pin "1")
+    (instances
+      (project "MiniAvionics"
+        (path "/db07439e-b2f9-4de9-a6da-003465a4a615/c809a2a1-09f7-4dc3-8e0e-630961f558de"
+          (reference "#PWR07") (unit 1)
+        )
+      )
+    )
+  )
+  (symbol (lib_id "power:VDD") (at 81.28 64.77 0) (unit 1)
+    (in_bom yes) (on_board yes) (dnp no)
+    (property "Reference" "#PWR08" (at 81.28 68.58 0)
+      (effects (font (size 1.27 1.27)) hide)
+    )
+    (property "Value" "VDD" (at 81.28 60.96 90)
+      (effects (font (size 1.27 1.27)) (justify left) hide)
+    )
+    (property "Footprint" "" (at 81.28 64.77 0)
+      (effects (font (size 1.27 1.27)) hide)
+    )
+    (property "Datasheet" "" (at 81.28 64.77 0)
+      (effects (font (size 1.27 1.27)) hide)
+    )
+    (pin "1")
+    (instances
+      (project "MiniAvionics"
+        (path "/db07439e-b2f9-4de9-a6da-003465a4a615/c809a2a1-09f7-4dc3-8e0e-630961f558de"
+          (reference "#PWR08") (unit 1)
+        )
+      )
+    )
+  )
   (symbol (lib_id "power:GND") (at 26.67 48.26 0) (unit 1)
     (in_bom yes) (on_board yes) (dnp no)
@@
       (effects (font (size 1.524 1.524)))
     )
-    (property "Footprint" "LGA10_BMP390_BOS" (at 40.64 40.64 0)
+    (property "Footprint" "MiniAvionics:LGA10_BMP390_BOS" (at 40.64 40.64 0)
       (effects (font (size 1.27 1.27) italic) hide)
     )
@@
     (pin "10")
     (pin "2")
-    (pin "3")
     (pin "4")
     (pin "5")
     (pin "6")
     (pin "7")
+    (pin "3")
     (pin "8")
     (pin "9")
@@
         )
       )
+    )
+  )
+  (symbol (lib_id "power:PWR_FLAG") (at 72.39 67.31 0) (unit 1)
+    (in_bom yes) (on_board yes) (dnp no) (fields_autoplaced)
+    (property "Reference" "#FLG01" (at 72.39 65.405 0)
+      (effects (font (size 1.27 1.27)) hide)
+    )
+    (property "Value" "PWR_FLAG" (at 72.39 62.23 0)
+      (effects (font (size 1.27 1.27)))
+    )
+    (property "Footprint" "" (at 72.39 67.31 0)
+      (effects (font (size 1.27 1.27)) hide)
+    )
+    (property "Datasheet" "~" (at 72.39 67.31 0)
+      (effects (font (size 1.27 1.27)) hide)
+    )
+    (pin "1")
+    (instances
+      (project "MiniAvionics"
+        (path "/db07439e-b2f9-4de9-a6da-003465a4a615/c809a2a1-09f7-4dc3-8e0e-630961f558de"
+          (reference "#FLG01") (unit 1)
+        )
+      )

Commit message: BMP 390 Schematic
Parts:
- added J1: 826629-4, CON4_1X4_P100UM_HDR2_TYC, symbol LSM9DS1:826629-4
- U1: footprint MiniAvionics:LGA10_BMP390_BOS -> MiniAvionics:LGA10_BMP390_BOS-M
Connections:
- net GND: now also J1.2
- new net SDI: J1.3
- new net SDO / INT: J1.4
- new net VDDIO* / VDD: J1.1
Changed lines of the file:
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@@
     (stroke (width 0) (type default))
+  )
+  (label "SDI" (at 49.53 68.58 180) (fields_autoplaced)
+    (effects (font (size 1.27 1.27)) (justify right bottom))
   )
   (label "VDDIO" (at 40.64 30.48 90) (fields_autoplaced)
     (effects (font (size 1.27 1.27)) (justify left bottom))
   )
-  (label "VDDIO" (at 81.28 64.77 90) (fields_autoplaced)
+  (label "VDDIO" (at 87.63 63.5 90) (fields_autoplaced)
     (effects (font (size 1.27 1.27)) (justify left bottom))
   )
@@
     (effects (font (size 1.27 1.27)) (justify left bottom))
   )
+  (label "SDO {slash} INT" (at 49.53 71.12 180) (fields_autoplaced)
+    (effects (font (size 1.27 1.27)) (justify right bottom))
+  )
   (label "SDA" (at 38.1 50.8 270) (fields_autoplaced)
+    (effects (font (size 1.27 1.27)) (justify right bottom))
+  )
+  (label "VDDIO* {slash} VDD" (at 49.53 63.5 180) (fields_autoplaced)
     (effects (font (size 1.27 1.27)) (justify right bottom))
   )
@@
     (effects (font (size 1.27 1.27)) (justify left bottom))
   )
+  (label "GND" (at 49.53 66.04 180) (fields_autoplaced)
+    (effects (font (size 1.27 1.27)) (justify right bottom))
+  )
   (symbol (lib_id "Device:LED") (at 99.06 39.37 90) (unit 1)
     (in_bom yes) (on_board yes) (dnp no)
@@
     )
   )
-  (symbol (lib_id "power:PWR_FLAG") (at 81.28 64.77 180) (unit 1)
+  (symbol (lib_id "power:PWR_FLAG") (at 87.63 63.5 180) (unit 1)
     (in_bom yes) (on_board yes) (dnp no) (fields_autoplaced)
-    (property "Reference" "#FLG02" (at 81.28 66.675 0)
-      (effects (font (size 1.27 1.27)) hide)
-    )
-    (property "Value" "PWR_FLAG" (at 81.28 69.85 0)
-      (effects (font (size 1.27 1.27)))
-    )
-    (property "Footprint" "" (at 81.28 64.77 0)
-      (effects (font (size 1.27 1.27)) hide)
-    )
-    (property "Datasheet" "~" (at 81.28 64.77 0)
+    (property "Reference" "#FLG02" (at 87.63 65.405 0)
+      (effects (font (size 1.27 1.27)) hide)
+    )
+    (property "Value" "PWR_FLAG" (at 87.63 68.58 0)
+      (effects (font (size 1.27 1.27)))
+    )
+    (property "Footprint" "" (at 87.63 63.5 0)
+      (effects (font (size 1.27 1.27)) hide)
+    )
+    (property "Datasheet" "~" (at 87.63 63.5 0)
       (effects (font (size 1.27 1.27)) hide)
     )
@@
         (path "/db07439e-b2f9-4de9-a6da-003465a4a615/c809a2a1-09f7-4dc3-8e0e-630961f558de"
           (reference "#FLG02") (unit 1)
+        )
+      )
+    )
+  )
+  (symbol (lib_id "LSM9DS1:826629-4") (at 49.53 63.5 0) (unit 1)
+    (in_bom yes) (on_board yes) (dnp no)
+    (property "Reference" "J1" (at 66.04 73.66 90)
+      (effects (font (size 1.524 1.524)) (justify left))
+    )
+    (property "Value" "826629-4" (at 63.5 73.66 90)
+      (effects (font (size 1.524 1.524)) (justify left))
+    )
+    (property "Footprint" "CON4_1X4_P100UM_HDR2_TYC" (at 49.53 63.5 0)
+      (effects (font (size 1.27 1.27) italic) hide)
+    )
+    (property "Datasheet" "826629-4" (at 49.53 63.5 0)
+      (effects (font (size 1.27 1.27) italic) hide)
+    )
+    (pin "1")
+    (pin "2")
+    (pin "3")
+    (pin "4")
+    (instances
+      (project "newlsm9ds1"
+        (path "/06f791fb-f574-4574-a583-188376710421"
+          (reference "J1") (unit 1)
+        )
+      )
+      (project "MiniAvionics"
+        (path "/db07439e-b2f9-4de9-a6da-003465a4a615/c809a2a1-09f7-4dc3-8e0e-630961f558de"
+          (reference "J1") (unit 1)
         )
       )
@@
     )
   )
-  (symbol (lib_id "power:GND") (at 72.39 67.31 0) (unit 1)
+  (symbol (lib_id "power:GND") (at 78.74 66.04 0) (unit 1)
     (in_bom yes) (on_board yes) (dnp no) (fields_autoplaced)
-    (property "Reference" "#PWR07" (at 72.39 73.66 0)
-      (effects (font (size 1.27 1.27)) hide)
-    )
-    (property "Value" "GND" (at 72.39 72.39 0)
-      (effects (font (size 1.27 1.27)))
-    )
-    (property "Footprint" "" (at 72.39 67.31 0)
-      (effects (font (size 1.27 1.27)) hide)
-    )
-    (property "Datasheet" "" (at 72.39 67.31 0)
+    (property "Reference" "#PWR07" (at 78.74 72.39 0)
+      (effects (font (size 1.27 1.27)) hide)
+    )
+    (property "Value" "GND" (at 78.74 71.12 0)
+      (effects (font (size 1.27 1.27)))
+    )
+    (property "Footprint" "" (at 78.74 66.04 0)
+      (effects (font (size 1.27 1.27)) hide)
+    )
+    (property "Datasheet" "" (at 78.74 66.04 0)
       (effects (font (size 1.27 1.27)) hide)
     )
@@
     )
   )
-  (symbol (lib_id "power:VDD") (at 81.28 64.77 0) (unit 1)
-    (in_bom yes) (on_board yes) (dnp no)
-    (property "Reference" "#PWR08" (at 81.28 68.58 0)
-      (effects (font (size 1.27 1.27)) hide)
-    )
-    (property "Value" "VDD" (at 81.28 60.96 90)
+  (symbol (lib_id "power:VDD") (at 87.63 63.5 0) (unit 1)
+    (in_bom yes) (on_board yes) (dnp no)
+    (property "Reference" "#PWR08" (at 87.63 67.31 0)
+      (effects (font (size 1.27 1.27)) hide)
+    )
+    (property "Value" "VDD" (at 87.63 59.69 90)
       (effects (font (size 1.27 1.27)) (justify left) hide)
     )
-    (property "Footprint" "" (at 81.28 64.77 0)
-      (effects (font (size 1.27 1.27)) hide)
-    )
-    (property "Datasheet" "" (at 81.28 64.77 0)
+    (property "Footprint" "" (at 87.63 63.5 0)
+      (effects (font (size 1.27 1.27)) hide)
+    )
+    (property "Datasheet" "" (at 87.63 63.5 0)
       (effects (font (size 1.27 1.27)) hide)
     )
@@
       (effects (font (size 1.524 1.524)))
     )
-    (property "Footprint" "MiniAvionics:LGA10_BMP390_BOS" (at 40.64 40.64 0)
+    (property "Footprint" "MiniAvionics:LGA10_BMP390_BOS-M" (at 40.64 40.64 0)
       (effects (font (size 1.27 1.27) italic) hide)
     )
@@
     )
   )
-  (symbol (lib_id "power:PWR_FLAG") (at 72.39 67.31 0) (unit 1)
+  (symbol (lib_id "power:PWR_FLAG") (at 78.74 66.04 0) (unit 1)
     (in_bom yes) (on_board yes) (dnp no) (fields_autoplaced)
-    (property "Reference" "#FLG01" (at 72.39 65.405 0)
-      (effects (font (size 1.27 1.27)) hide)
-    )
-    (property "Value" "PWR_FLAG" (at 72.39 62.23 0)
-      (effects (font (size 1.27 1.27)))
-    )
-    (property "Footprint" "" (at 72.39 67.31 0)
-      (effects (font (size 1.27 1.27)) hide)
-    )
-    (property "Datasheet" "~" (at 72.39 67.31 0)
-      (effects (font (size 1.27 1.27)) hide)
-    )
+    (property "Reference" "#FLG01" (at 78.74 64.135 0)
+      (effects (font (size 1.27 1.27)) hide)
+    )
+    (property "Value" "PWR_FLAG" (at 78.74 60.96 0)
+      (effects (font (size 1.27 1.27)))
+    )
+    (property "Footprint" "" (at 78.74 66.04 0)
+      (effects (font (size 1.27 1.27)) hide)
+    )
+    (property "Datasheet" "~" (at 78.74 66.04 0)
+      (effects (font (size 1.27 1.27)) hide)
+    )

Commit message: finished bmp
Parts:
- U1: footprint MiniAvionics:LGA10_BMP390_BOS-M -> MiniAvionics:LGA10_BMP390_BOS-L
Connections:
- net SDI is gone; now on net SDA: J1.3
- net SDO / INT is gone; now on net GND: J1.4
- net VDDIO* is gone; now on net VDD: U1.6 (CSB)
- net VDDIO* / VDD is gone; now on net VDD: J1.1
- net GND: no longer J1.2
- net I2C_PS: now also J1.2
- no-connect marks 5 -> 2
Changed lines of the file:
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@@
   (junction (at 40.64 35.56) (diameter 0) (color 0 0 0 0)
   )
+  (junction (at 82.55 58.42) (diameter 0) (color 0 0 0 0)
+  )
   (junction (at 91.44 43.18) (diameter 0) (color 0 0 0 0)
   )
@@
   )
   (no_connect (at 81.28 48.26))
-  (no_connect (at 38.1 50.8))
   (no_connect (at 36.83 43.18))
-  (no_connect (at 40.64 50.8))
-  (no_connect (at 81.28 50.8))
   (wire (pts (xy 40.64 30.48) (xy 40.64 35.56))
     (stroke (width 0) (type default))
   )
+  (wire (pts (xy 38.1 68.58) (xy 49.53 68.58))
+    (stroke (width 0) (type default))
+  )
+  (wire (pts (xy 82.55 58.42) (xy 106.68 58.42))
+    (stroke (width 0) (type default))
+  )
+  (wire (pts (xy 49.53 58.42) (xy 49.53 63.5))
+    (stroke (width 0) (type default))
+  )
   (wire (pts (xy 26.67 45.72) (xy 40.64 45.72))
     (stroke (width 0) (type default))
   )
+  (wire (pts (xy 82.55 50.8) (xy 81.28 50.8))
+    (stroke (width 0) (type default))
+  )
   (wire (pts (xy 39.37 39.37) (xy 33.02 39.37))
     (stroke (width 0) (type default))
@@
     (stroke (width 0) (type default))
   )
-  (wire (pts (xy 38.1 48.26) (xy 38.1 50.8))
+  (wire (pts (xy 38.1 48.26) (xy 38.1 68.58))
     (stroke (width 0) (type default))
   )
@@
     (stroke (width 0) (type default))
   )
+  (wire (pts (xy 40.64 50.8) (xy 40.64 66.04))
+    (stroke (width 0) (type default))
+  )
+  (wire (pts (xy 40.64 66.04) (xy 49.53 66.04))
+    (stroke (width 0) (type default))
+  )
   (wire (pts (xy 38.1 48.26) (xy 40.64 48.26))
     (stroke (width 0) (type default))
@@
     (stroke (width 0) (type default))
   )
+  (wire (pts (xy 91.44 25.4) (xy 91.44 27.94))
+    (stroke (width 0) (type default))
+  )
+  (wire (pts (xy 106.68 25.4) (xy 106.68 58.42))
+    (stroke (width 0) (type default))
+  )
   (wire (pts (xy 81.28 45.72) (xy 91.44 45.72))
     (stroke (width 0) (type default))
   )
+  (wire (pts (xy 49.53 58.42) (xy 82.55 58.42))
+    (stroke (width 0) (type default))
+  )
   (wire (pts (xy 81.28 40.64) (xy 86.36 40.64))
     (stroke (width 0) (type default))
   )
+  (wire (pts (xy 91.44 25.4) (xy 106.68 25.4))
+    (stroke (width 0) (type default))
+  )
   (wire (pts (xy 86.36 31.75) (xy 91.44 31.75))
     (stroke (width 0) (type default))
@@
     (stroke (width 0) (type default))
   )
+  (wire (pts (xy 82.55 50.8) (xy 82.55 58.42))
+    (stroke (width 0) (type default))
+  )
   (wire (pts (xy 91.44 43.18) (xy 91.44 45.72))
     (stroke (width 0) (type default))
@@
     (stroke (width 0) (type default))
   )
-  (label "SDI" (at 49.53 68.58 180) (fields_autoplaced)
+  (label "SDA" (at 49.53 68.58 180) (fields_autoplaced)
     (effects (font (size 1.27 1.27)) (justify right bottom))
   )
@@
     (effects (font (size 1.27 1.27)) (justify left bottom))
   )
-  (label "SDO {slash} INT" (at 49.53 71.12 180) (fields_autoplaced)
+  (label "SDO" (at 49.53 66.04 180) (fields_autoplaced)
     (effects (font (size 1.27 1.27)) (justify right bottom))
   )
@@
     (effects (font (size 1.27 1.27)) (justify right bottom))
   )
-  (label "VDDIO* {slash} VDD" (at 49.53 63.5 180) (fields_autoplaced)
+  (label "VDDIO" (at 49.53 63.5 180) (fields_autoplaced)
     (effects (font (size 1.27 1.27)) (justify right bottom))
   )
@@
     (effects (font (size 1.27 1.27)) (justify right bottom))
   )
-  (label "VDDIO*" (at 81.28 50.8 0) (fields_autoplaced)
-    (effects (font (size 1.27 1.27)) (justify left bottom))
-  )
-  (label "GND" (at 49.53 66.04 180) (fields_autoplaced)
+  (label "VDDIO" (at 82.55 50.8 180) (fields_autoplaced)
+    (effects (font (size 1.27 1.27)) (justify right bottom))
+  )
+  (label "GND" (at 49.53 71.12 180) (fields_autoplaced)
     (effects (font (size 1.27 1.27)) (justify right bottom))
   )
@@
       (effects (font (size 1.524 1.524)))
     )
-    (property "Footprint" "MiniAvionics:LGA10_BMP390_BOS-M" (at 40.64 40.64 0)
+    (property "Footprint" "MiniAvionics:LGA10_BMP390_BOS-L" (at 40.64 40.64 0)
       (effects (font (size 1.27 1.27) italic) hide)
     )
