File: hardware/MiniAvionics/MiniAvionics.kicad_pcb (KiCad board)
At the start: 2 copper layers, 7 parts, among them U1 BMP390

Commit message: finished bmp
Parts:
- added J1: 826629-4, MiniAvionics:CON4_1X4_P100UM_HDR2_TYC, F.Cu at (178.5, 99.2)
- U1: footprint MiniAvionics:LGA10_BMP390_BOS -> MiniAvionics:LGA10_BMP390_BOS-L
- moved R1 4.16 mm to (178.3, 91.5), turned to 180 degrees
- moved R3 3.18 mm to (185.7, 95.5)
- moved GREEN1 3.11 mm to (186.9, 92.3), turned to -90 degrees
- moved C2 3.08 mm to (184.7, 92.3), turned to 90 degrees
- moved R2 1.50 mm to (177.6, 94.7)
- moved C1 1.29 mm to (181.6, 91.5), turned to 0 degrees
- moved U1 0.59 mm to (181.2, 95.0)
Connections:
- U1 pad 6: /BMP390/VDDIO* -> VDD
Routing:
- net GND: track 2.00 -> 26.7 mm, vias 0 -> 2
- net VDD: track 11.2 -> 27.9 mm
- net /BMP390/SDA: track 0.00 -> 11.7 mm, vias 0 -> 2
- net /BMP390/I2C_PS: track 0.00 -> 5.76 mm, vias 0 -> 2
- net /BMP390/SCL: track 0.00 -> 3.51 mm
- net Net-(GREEN1-A): track 0.00 -> 2.61 mm
- added copper zone on B.Cu, net GND
- added copper zone on F.Cu, net VDD
Other:
- board outline added: 12.9 x 11.1 mm
