File: hardware/MiniAvionics/newlsm9ds1.kicad_pcb (KiCad board)
At the start: 2 copper layers, 13.8 x 19.4 mm, 17 parts, among them IC1 LSM9DS1, J1 826629-4

Commit message: Procrastinated PRISM commit
Changed lines of the file:
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@@
       (outputformat 1)
       (mirror false)
-      (drillshape 1)
+      (drillshape 0)
       (scaleselection 1)
       (outputdirectory "")
@@
     (fp_line (start 1.5 0.85) (end -1.3 0.85)
       (stroke (width 0.1) (type solid)) (layer "F.Fab"))
-    (pad "1" smd roundrect (at -1.5 -0.05) (size 0.75 0.8) (layers "F.Cu" "F.Paste" "F.Mask") (roundrect_rratio 0.2272727273)
+    (pad "1" smd roundrect (at -1.5 -0.05) (size 0.75 0.8) (layers "F.Cu" "F.Paste" "F.Mask") (roundrect_rratio 0.2272733333)
       (net 5 "/CS_A{slash}G") (pinfunction "A") (pintype "passive"))
-    (pad "2" smd roundrect (at 1.7 -0.05 180) (size 0.75 0.8) (layers "F.Cu" "F.Paste" "F.Mask") (roundrect_rratio 0.2272727273)
+    (pad "2" smd roundrect (at 1.7 -0.05 180) (size 0.75 0.8) (layers "F.Cu" "F.Paste" "F.Mask") (roundrect_rratio 0.2272733333)
       (net 14 "Net-(D2-C)") (pinfunction "C") (pintype "passive"))
   )
@@
     (fp_line (start 1.5 0.85) (end -1.3 0.85)
       (stroke (width 0.1) (type solid)) (layer "F.Fab"))
-    (pad "1" smd roundrect (at -1.5 -0.05) (size 0.75 0.8) (layers "F.Cu" "F.Paste" "F.Mask") (roundrect_rratio 0.2272727273)
+    (pad "1" smd roundrect (at -1.5 -0.05) (size 0.75 0.8) (layers "F.Cu" "F.Paste" "F.Mask") (roundrect_rratio 0.2272733333)
       (net 6 "/CS_M") (pinfunction "A") (pintype "passive"))
-    (pad "2" smd roundrect (at 1.7 -0.05 180) (size 0.75 0.8) (layers "F.Cu" "F.Paste" "F.Mask") (roundrect_rratio 0.2272727273)
+    (pad "2" smd roundrect (at 1.7 -0.05 180) (size 0.75 0.8) (layers "F.Cu" "F.Paste" "F.Mask") (roundrect_rratio 0.2272733333)
       (net 13 "Net-(D1-C)") (pinfunction "C") (pintype "passive"))
   )
