File: hardware/_REV3_FALL_2023/PRISM_Teensy/board_one_teensy_22/board_one_teensy_22.kicad_pcb (KiCad board)
At the start: 2 copper layers, 61 x 88.9 mm, 26 parts, among them J1 Micro_SD_Card_Det_Hirose_DM3AT, J3 3387, U1 Teensy4.0, U3 3966, U4 RFM69HCW_Breakout, U5 SFN-1407PA7.6

Commit message: Final PRISM FC Board
Parts:
- GPS1: footprint Connector_JST:JST_XH_B2B-XH-A_1x02_P2.50mm_Vertical -> Connector_PinHeader_2.54mm:PinHeader_1x02_P2.54mm_Vertical
- Power1: footprint Connector_JST:JST_XH_B4B-XH-A_1x04_P2.50mm_Vertical -> Connector_PinHeader_2.54mm:PinHeader_1x04_P2.54mm_Vertical
- Pyro1, Stepper1: footprint Connector_JST:JST_XH_B5B-XH-A_1x05_P2.50mm_Vertical -> Connector_PinHeader_2.54mm:PinHeader_1x05_P2.54mm_Vertical
- moved GPS1 133.1 mm to (110.7, 105.7)
- moved C1 130.4 mm to (112.8, 112.7), turned to 180 degrees
- moved Power1 129.4 mm to (110.7, 92.2)
- moved R4 129.2 mm to (112.8, 114.5)
- moved R5 129.2 mm to (112.8, 116.1), turned to 180 degrees
- moved D3 126.2 mm to (122.0, 108.4)
- moved C2 125.7 mm to (116.8, 108.3), turned to -90 degrees
- moved H1 125.4 mm to (118.6, 53.3)
- moved U5 124.2 mm to (120.3, 66.3), turned to 90 degrees
- moved H3 120.4 mm to (118.6, 135.8)
- moved Pyro1 112.9 mm to (110.8, 60.1)
- moved Stepper1 112.4 mm to (110.8, 76.0)
- moved D5 111.1 mm to (136.7, 108.5)
- moved R1 97.4 mm to (147.0, 123.5), turned to 180 degrees
- moved C3 96.3 mm to (147.6, 117.9), turned to -90 degrees
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Connections:
- U1 pad 1: /PYRO 1 -> /CONT 1
- U1 pad 2: /PYRO 2 -> /CONT 2
- U1 pad 3: /CONT 1 -> /PYRO 1
- U1 pad 4: /CONT 2 -> /PYRO 2
Routing:
- net GND: track 0.00 -> 327.7 mm, vias 0 -> 4
- net /3.3V: track 0.00 -> 185.0 mm, vias 0 -> 2
- net /5V: track 0.00 -> 122.8 mm
- net /V_Mon: track 0.00 -> 120.8 mm, vias 0 -> 4
- net /SD_DETECT: track 0.00 -> 100.4 mm, vias 0 -> 3
- net /SCL: track 0.00 -> 98.0 mm, vias 0 -> 6
- net /SDA: track 0.00 -> 97.1 mm, vias 0 -> 8
- net /SD_CS: track 0.00 -> 96.7 mm
- net /RX 5: track 0.00 -> 87.1 mm
- net /MOSI: track 0.00 -> 81.7 mm, vias 0 -> 7
- net /MISO: track 0.00 -> 81.5 mm, vias 0 -> 8
- net /SD_SCK: track 0.00 -> 77.1 mm, vias 0 -> 4
- net /Radio_RST: track 0.00 -> 67.6 mm
- net /EN: track 0.00 -> 53.7 mm
- net /ARM: track 0.00 -> 53.6 mm
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- added copper zone on F.Cu, net /3.3V
Other:
- outline, holes or cut-outs redrawn
- board text added: "9-Axis IMU"
- board text added: "Barometer"
- board text added: "Buzzer"
- board text added: "GND VB 5V 3V3"
- board text added: "GPS"
- board text added: "Micro-SD"
- board text added: "P2 P1 C2 C1 A"
- board text added: "Power"
- board text added: "Pyro"
- board text added: "Radio"
- board text added: "Raveionics"
- board text added: "SDA SCL"
- board text added: "ST DR EN TX RX"
- board text added: "Stepper"
- board text added: "Teensy 4.0"
