File: hardware/_REV3_FALL_2023/PRISM_Teensy w GPS/board_one_teensy_22/board_one_teensy_22.kicad_pcb (KiCad board)
At the start: 2 copper layers, 61 x 88.9 mm, 33 parts, among them J1 Micro_SD_Card_Det_Hirose_DM3AT, J3 3387, Q1 AO3400A, Q2 AO3400A, U1 Teensy4.0, U2 GPS-14414, U3 3966, U4 RFM69HCW_Breakout, U5 CT25E-16T150-1, U6 CMI-9605-1280T

Commit message: Final FC Board
Parts:
- moved C1 29.1 mm to (115.3, 106.9), turned to -90 degrees
- moved C4 14.1 mm to (154.7, 94.5), turned to 180 degrees
- moved R4 3.13 mm to (139.0, 92.7)
- moved R5 3.13 mm to (139.0, 91.2)
- moved U6 1.27 mm to (120.1, 102.1)
- moved D3 0.38 mm to (151.0, 90.4)
- moved D5 0.38 mm to (158.6, 90.4)
Routing:
- net /SD_DETECT: track 120.6 -> 68.8 mm, vias 6 -> 5
- net GND: track 258.9 -> 283.9 mm, vias 6 -> 10
- net /SDA: track 115.4 -> 98.4 mm, vias 7 -> 2
- net /SCL: track 106.7 -> 89.9 mm, vias 6 -> 1
- net /5V: track 138.9 -> 147.7 mm
- net /V_Mon: track 33.1 -> 39.3 mm
- net /VBAT: track 73.7 -> 78.3 mm, vias 0 -> 2
- net /Radio_RST: track 45.3 -> 42.0 mm
- net /NEOPIXEL: track 8.17 -> 11.2 mm
- net /CS 1: track 42.9 -> 40.3 mm
- net /RX 5: track 30.5 -> 29.0 mm
- net /3.3V: track 163.1 -> 161.8 mm, vias 8 -> 9
- net /CONT 1: track 44.7 -> 45.9 mm, vias 4 -> 2
- net /PYRO 2: track 89.2 -> 88.0 mm
- net /ARM: track 48.5 -> 49.6 mm, vias 4 -> 2
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Other:
- board text added: "GND 3V VB 5V"
- board text added: "Lili Baker"
- board text removed: "GND VB 5V"
