File: hardware/Certification_Avionics/Certification_Avionics.kicad_sch (KiCad schematic)
At the start: 66 parts, among them J1 2 Pin Connector, J2 2 Pin Connector, J3 2 Pin Connector, J4 2 Pin Connector, J5 USB_Micro_B, SW1 SW, SW2 SW, SW3 SW_DIP_x01, U1 ESP32-S3-WROOM-1-N16R8, U2 LED_DRIVER, U3 LED_DRIVER, U4 BMS, U5 Voltage Regulator

Commit message: Add comments to cert avionics
Parts:
- added R36: 24k, symbol Device:R
- added SW6: SW_DIP_x01, symbol Switch:SW_DIP_x01
- C6, C7: value 100n -> 100u
- R25: value 12k -> 24k
- U5: Digikey (none) -> https://www.digikey.com/en/products/detail/microchip-techno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
- renumbered SW3 to SW4, SW3 to SW5
Connections:
- net EN: no longer C3.1
- net GND: now also R36.1
- net ISET: now also SW6.1
- net VBAT: now also R28.1
- net VCC: now reaches C13.1, U4.4 (VCC)
- net VCC: now also U4.8 (NTC)
- net at C10.1, C9.1, U4.11 (SYS): now also C3.1
- net VBAT1 renamed VPYRO
- net VPYRO: no longer R28.1
- new net: R36.2, SW6.2
- no-connect marks 8 -> 7
Other:
- added sheet Checklist (checklist.kicad_sch)
- sheet Sensors & Pinouts: file untitled.kicad_sch -> sensors.kicad_sch
- note added: "1/3 divider Vin,max = 8.4V Vout,max = 2.8V"
- note added: "IDK how to find this"
- note added: "Icc = 24kOhm/Riset = 0.5A"
- note added: "Page 20 ->"
- note added: "Page 35 -> Rl = 10k Rh = 27.5k Vin,min = 1.2V*(Rh+Rl)/Rl = 4.5V"
- note added: "Page 36 ->"
- note added: "Page 36 Selecting the System Capacitor"
- note added: "Vdim,min = 0.3V 8k/(200k+8k)*5V = 0.192V"
- note added: "^ Page 36"
- moved on the sheet: C1, C11, C12, C2, C4, C5, L3, R10, R2, R21, R23, R24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
